Commit message: Cheetah simulation part.2

File: examples/cheetah/cheetah/urdf/cheetah.urdf (robot description, URDF)
Before this commit: robot cheetah, 17 links, 17 joints
Links:
- added link ground
Joints:
- removed joint trunk_to_trunk_inertia_floating
- added joint ground_t_floating: type revolute, parent ground, child trunk, origin xyz=0 0 0 rpy=0 0 0, limit lower=-0.872664625997 upper=1.0471975512 effort=20 velocity=10.6

Commit message: Cheetah update and small fixes

File: examples/cheetah/cheetah/urdf/cheetah.urdf (robot description, URDF)
Before this commit: robot cheetah, 18 links, 17 joints
Joints:
- joint ground_t_floating: origin xyz=0 0 0 rpy=0 0 0 -> xyz=0 0 0.45 rpy=0 0 0
