Commit message: Minor fixes to Chain and URDF parser

File: examples/iiwa/iiwa14.urdf (robot description, URDF)
Before this commit: robot iiwa14, 11 links, 10 joints
Links:
- removed link base
- link iiwa_link_0: geometry collision cylinder length=0.17 radius=0.139; visual mesh filename=meshes/visual/link_0.stl
- link iiwa_link_1: geometry collision cylinder length=0.29 radius=0.101; visual mesh filename=meshes/visual/link_1.stl
- link iiwa_link_2: geometry collision cylinder length=0.29 radius=0.101; visual mesh filename=meshes/visual/link_2.stl
- link iiwa_link_3: geometry collision cylinder length=0.29 radius=0.092; visual mesh filename=meshes/visual/link_3.stl
- link iiwa_link_4: geometry collision cylinder length=0.25 radius=0.092; visual mesh filename=meshes/visual/link_4.stl
- link iiwa_link_5: geometry collision cylinder length=0.29 radius=0.07; visual mesh filename=meshes/visual/link_5.stl
- link iiwa_link_6: geometry collision mesh filename=meshes/collision/link_6.stl; visual mesh filename=meshes/visual/link_6.stl
- link iiwa_link_7: geometry collision mesh filename=meshes/collision/link_7.stl; visual mesh filename=meshes/visual/link_7.stl
Joints:
- removed joint base_joint

Commit message: Fixed iiwa base

File: examples/iiwa/iiwa14.urdf (robot description, URDF)
Before this commit: robot iiwa14, 10 links, 9 joints
Links:
- added link base
Joints:
- added joint base_to_0: type fixed, parent base, child iiwa_link_0, origin xyz=0 0 0 rpy=0 0 0
