Commit message: a1 bullet simulation

File: examples/a1/urdf/a1.urdf (robot description, URDF)
Before this commit: robot a1_description, 19 links, 18 joints
Links:
- removed link ground
- added link base; visual box size=0.001 0.001 0.001
Joints:
- removed joint ground_t_floating
- added joint floating_base_floating: type fixed, parent base, child trunk, origin xyz=0 0 0 rpy=0 0 0
